File: Boards/Avionics/HYDRA_V2/HYDRA_V2/HYDRA_V2.kicad_sch (KiCad schematic)
At the start: 38 parts, among them IC1 MAX31855KASA+T, IC2 MAX31855KASA+T, IC3 MAX31855KASA+T, J1 1723103102, J2 1723103102, J3 1723103102, J4 1723103102, J5 1723103103, J6 1723103103, Q1 IRLB3813PBF-ND, Q2 IRLB3813PBF-ND, Q3 IRLB3813PBF-ND, U1 MAX485_MODULE_5V_LOGIC_TLL_TO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, U3 ThermoConnector, U4 ThermoConnector, U5 ThermoConnector

Commit message: Hydra V2
Parts:
- added C4: 0.1uF, symbol Device:C_Small
- added C5: C_Small, symbol Device:C_Small
- added D7, D8: 1N5817, Diode_THT:D_DO-41_SOD81_P10.16mm_Horizontal, symbol Diode:1N5817
- added J8: 1723163304, 1723163304:MOLEX_1723163304, symbol 1723163304:1723163304
- added Q4, Q5, Q6, Q7: IRLB3813PBF-ND, Package_TO_SOT_THT:TO-220-3_Vertical, symbol Transistor_FET:IRLB8721PBF
- added Q8: Q_NPN_BCE, symbol Transistor_BJT:Q_NPN_BCE
- added R10, R11, R12, R13, R14, R9: 10K, symbol Device:R
Connections:
- net +12V: now also J1.1, J2.1, J3.1, D7.1 (K), D8.1 (K), J8.1, Q7.2 (D), R11.1; no longer J1.4 (SHIELD2), J2.4 (SHIELD2), J3.4 (SHIELD2)
- net +3.3V: now also R13.1
- net +5V: now also C4.1, C5.1
- net GND: now also J1.3 (SHIELD1), J1.4 (SHIELD2), J2.3 (SHIELD1), J2.4 (SHIELD2), J3.3 (SHIELD1), J3.4 (SHIELD2), C4.2, C5.2, J8.2, J8.4, Q4.3 (S), Q5.3 (S), Q8.3 (E), R10.2, R11.2, R12.2, R9.2; no longer J1.1, J1.2, J2.1, J2.2, J3.1, J3.2
- net at D2.2 (A), Q2.2 (D): now also J2.2; no longer J2.3 (SHIELD1)
- net at D3.2 (A), Q3.2 (D): now also J3.2; no longer J3.3 (SHIELD1)
- net at D1.2 (A), Q1.2 (D): now also J1.2; no longer J1.3 (SHIELD1)
- new net: Q5.1 (G), R10.1
- new net: D8.2 (A), Q5.2 (D)
- new net: J8.3, Q7.3 (S), R12.1
- new net: Q4.1 (G), R9.1
- new net: D7.2 (A), Q4.2 (D)
- new net: Q8.1 (B), R14.2
- new net SBALL_1: R14.1
- new net SBALL_CLOSE_1: Q7.1 (G), Q8.2 (C), R13.2
Other:
- moved on the sheet: D1, D2, D3, J1, J2, J3, J4, Q1, Q2, Q3, R1, R2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
