File: Boards/Avionics/HYDRA_V2/HYDRA_V2/HYDRA_V2.kicad_sch (KiCad schematic)
At the start: 57 parts, among them IC1 MAX31855KASA+T, IC2 MAX31855KASA+T, IC3 MAX31855KASA+T, IC4 SP3485CN-L_TR, J4 1723103102, J5 1723103103, J6 1723103103, Q1 PMOS, Q14 PMOS, Q15 IRLB3813PBF-ND, Q16 IRLB3813PBF-ND, Q17 PMOS, Q2 IRLB3813PBF-ND, Q4 IRLB3813PBF-ND, Q5 PMOS, Q6 IRLB3813PBF-ND, Q7 PMOS, Q8 IRLB3813PBF-ND, Q9 PMOS, U3 ThermoConnector, U4 ThermoConnector, U5 ThermoConnector

Commit message: Hydra v2
Parts:
- removed U6, U7, U8: ~, DCDCModule:DCDC_Module, symbol Mini Dc-Dc:MiniDCDCBoost
- added C10, C17, C26, C35: 2.7nF, Capacitor_SMD:C_0603_1608Metric_Pad1.08x0.95mm_HandSolder, symbol Device:C_Small
- added C11, C20, C29, C38: 22pF, Capacitor_SMD:C_0603_1608Metric_Pad1.08x0.95mm_HandSolder, symbol Device:C_Small
- added C12, C13, C14, C21, C22, C23, C30, C31, C32, C39, C40, C41: 22uF, Capacitor_SMD:C_0603_1608Metric_Pad1.08x0.95mm_HandSolder, symbol Device:C_Small
- added C15, C24, C33, C6: 10uF, Capacitor_SMD:C_0805_2012Metric_Pad1.18x1.45mm_HandSolder, symbol Device:C_Small
- added C16, C25, C34, C7: 10nF, Capacitor_SMD:C_0603_1608Metric_Pad1.08x0.95mm_HandSolder, symbol Device:C_Small
- added C18, C27, C36, C8: 100nF, Capacitor_SMD:C_0603_1608Metric_Pad1.08x0.95mm_HandSolder, symbol Device:C_Small
- added C19, C28, C37, C9: 47pF, Capacitor_SMD:C_0603_1608Metric_Pad1.08x0.95mm_HandSolder, symbol Device:C_Small
- added D7: LED, LED_THT:LED_D3.0mm, symbol Device:LED
- added L1, L2, L3, L4: 6.8uH, SPM10054T-6R8M-HZR:SPM10054T6R8MHZR, symbol Device:L_Small
- added R12: 62, Resistor_SMD:R_0805_2012Metric, symbol Device:R
- added R13, R19, R27, R30: 27kO, Resistor_SMD:R_0603_1608Metric_Pad0.98x0.95mm_HandSolder, symbol Device:R_Small
- added R14, R28, R31: 210kO, Resistor_SMD:R_0603_1608Metric_Pad0.98x0.95mm_HandSolder, symbol Device:R_Small
- added R18, R26, R29, R32: 22.1kO, Resistor_SMD:R_0603_1608Metric_Pad0.98x0.95mm_HandSolder, symbol Device:R_Small
- added R25: 69.8kO, Resistor_SMD:R_0603_1608Metric_Pad0.98x0.95mm_HandSolder, symbol Device:R_Small
- added U1, U10, U11, U12: AP64501SP-13, AP64501SP_13:SOP_AP64501SP-13_DIO, symbol AP64501SP_13:AP64501SP-13
- Q1, Q14, Q17, Q5, Q7, Q9: footprint Package_TO_SOT_THT:TO-220-3_Vertical -> STD46P4LLF6:STD46P4LLF6
- Q15, Q16, Q2, Q4, Q6, Q8: footprint Package_TO_SOT_THT:TO-220-3_Vertical -> Package_TO_SOT_SMD:SOT-223
- U2: value ~ -> (none)
Connections:
- net +3.3V: now also D7.2 (A); no longer D6.2 (A)
- net +5V: now also D6.2 (A); no longer D5.2 (A)
- net GND: now also C10.2, C11.2, C12.2, C13.2, C14.2, C15.2, C16.2, C17.2, C20.2, C21.2, C22.2, C23.2, C24.2, C25.2, C26.2, C29.2, C30.2, C31.2, C32.2, C33.2, C34.2, C35.2, C38.2, C39.2, C40.2, C41.2, C6.2, C7.2, R12.2, R18.2, R26.2, R29.2, R32.2, U1.7 (GND), U1.EPAD, U10.7 (GND), U10.EPAD, U11.7 (GND), U11.EPAD, U12.7 (GND), U12.EPAD
- net VIN: now also C15.1, C24.1, C33.1, C6.1, U1.2 (VIN), U1.3 (EN), U10.2 (VIN), U10.3 (EN), U11.2 (VIN), U11.3 (EN), U12.2 (VIN), U12.3 (EN)
- net Servo_VCC renamed +8.4V
- net +8.4V: now also D5.2 (A), C12.1, C13.1, C14.1, C9.1, L1.2, R14.1
- new net: C36.1, U12.1 (BST)
- new net: C36.2, L4.1, U12.8 (SW)
- new net: C38.1, R30.1, U12.6 (COMP)
- new net: C35.1, R30.2
- new net: C37.2, R31.2, R32.1, U12.5 (FB)
- new net: D7.1 (K), R12.1
- new net: C28.1, C30.1, C31.1, C32.1, L3.2, R28.1
- new net: C26.1, R27.2
- new net: C37.1, C39.1, C40.1, C41.1, L4.2, R31.1
- new net: C8.1, U1.1 (BST)
- new net: C8.2, L1.1, U1.8 (SW)
- new net: C9.2, R14.2, R18.1, U1.5 (FB)
- new net: C29.1, R27.1, U11.6 (COMP)
- new net: C7.1, U1.4 (SS)
- new net: C11.1, R13.1, U1.6 (COMP)
- new net: C19.1, C21.1, C22.1, C23.1, L2.2, R25.1
- new net: C19.2, R25.2, R26.1, U10.5 (FB)
- new net: C10.1, R13.2
- new net: C28.2, R28.2, R29.1, U11.5 (FB)
- new net: C27.2, L3.1, U11.8 (SW)
- new net: C16.1, U10.4 (SS)
- new net: C18.1, U10.1 (BST)
- new net: C20.1, R19.1, U10.6 (COMP)
- new net: C18.2, L2.1, U10.8 (SW)
- new net: C17.1, R19.2
- new net: C27.1, U11.1 (BST)
- new net: C34.1, U12.4 (SS)
- new net: C25.1, U11.4 (SS)
Other:
- note added: "Buck Converter"
- note removed: "DC-DC Converter"
- moved on the sheet: D4, D5, D6, H1, H2, H3, H4, R6, R7, R8

Commit message: Hydra v2 almost done
Parts:
- removed C15: 10uF, Capacitor_SMD:C_0805_2012Metric_Pad1.18x1.45mm_HandSolder, symbol Device:C_Small
- removed C16: 10nF, Capacitor_SMD:C_0603_1608Metric_Pad1.08x0.95mm_HandSolder, symbol Device:C_Small
- removed C17: 2.7nF, Capacitor_SMD:C_0603_1608Metric_Pad1.08x0.95mm_HandSolder, symbol Device:C_Small
- removed C18: 100nF, Capacitor_SMD:C_0603_1608Metric_Pad1.08x0.95mm_HandSolder, symbol Device:C_Small
- removed C19: 47pF, Capacitor_SMD:C_0603_1608Metric_Pad1.08x0.95mm_HandSolder, symbol Device:C_Small
- removed C20: 22pF, Capacitor_SMD:C_0603_1608Metric_Pad1.08x0.95mm_HandSolder, symbol Device:C_Small
- removed C21, C22, C23: 22uF, Capacitor_SMD:C_0603_1608Metric_Pad1.08x0.95mm_HandSolder, symbol Device:C_Small
- removed L2: 6.8uH, SPM10054T-6R8M-HZR:SPM10054T6R8MHZR, symbol Device:L_Small
- removed Q1, Q14, Q17, Q5, Q7, Q9: PMOS, STD46P4LLF6:STD46P4LLF6, symbol Simulation_SPICE:PMOS
- removed Q2, Q4, Q6, Q8: IRLB3813PBF-ND, Package_TO_SOT_SMD:SOT-223, symbol Transistor_FET:IRLB8721PBF
- removed R1, R10, R11, R15, R16, R17, R2, R3, R4, R9: 10K, Resistor_SMD:R_0805_2012Metric_Pad1.20x1.40mm_HandSolder, symbol Device:R
- removed R19: 27kO, Resistor_SMD:R_0603_1608Metric_Pad0.98x0.95mm_HandSolder, symbol Device:R_Small
- removed R25: 69.8kO, Resistor_SMD:R_0603_1608Metric_Pad0.98x0.95mm_HandSolder, symbol Device:R_Small
- removed R26: 22.1kO, Resistor_SMD:R_0603_1608Metric_Pad0.98x0.95mm_HandSolder, symbol Device:R_Small
- removed U10: AP64501SP-13, AP64501SP_13:SOP_AP64501SP-13_DIO, symbol AP64501SP_13:AP64501SP-13
- added J1: XT30UPB-F, XT30UPB-F:XT30UPBF, symbol XT30UPB-F:XT30UPB-F
- added J10, J8, J9: 1723103103, 1723103103:MOLEX_1723103103, symbol 1723103103:1723103103
- added Q10, Q11, Q12, Q3, Q4, Q5: STD46P4LLF6, STD46P4LLF6, symbol STD46P4LLF6:STD46P4LLF6
- added Q17, Q18, Q19, Q20: IRLB3813PBF-ND, Package_TO_SOT_SMD:SOT-223, symbol Transistor_FET:IRLB8721PBF
- added R25, R26, R33, R34, R35, R36, R37, R38, R39, R40: 10K, Resistor_SMD:R_0805_2012Metric_Pad1.20x1.40mm_HandSolder, symbol Device:R
- C29: value 22pF -> 33pF
- C38: value 22pF -> 15pF
- D4, D5, D6, D7: footprint LED_THT:LED_D3.0mm -> LED-Yellow_VLMY1300-GS08:LEDC1608X100N
- R27: value 27kO -> 15.8kO
- R28: value 210kO -> 115.8kO
- R30: value 27kO -> 37.4kO
- R31: value 210kO -> 309kO
Connections:
- net +12V: now also C37.1, C39.1, C40.1, C41.1, L4.2, R31.1, Q10.3 (S), Q11.3 (S), Q12.3 (S), Q3.3 (S), Q4.3 (S), Q5.3 (S), R26.1, R34.1, R37.1, R39.1
- net +3.3V: now also A1.36 (3V3)
- net +5V: now also C28.1, C30.1, C31.1, C32.1, L3.2, R28.1
- net GND: now also J1.1, J10.2, J10.S1 (SHIELD1), J10.S2 (SHIELD2), J8.2, J8.S1 (SHIELD1), J8.S2 (SHIELD2), J9.2, J9.S1 (SHIELD1), J9.S2 (SHIELD2), Q17.3 (S), Q18.3 (S), Q19.3 (S), Q20.3 (S), R25.2, R33.2, R35.2, R36.2, R38.2, R40.2
- net RS_A: now also J4.4 (SHIELD2); no longer J4.3 (SHIELD1)
- net RS_B: now also J4.3 (SHIELD1); no longer J4.4 (SHIELD2)
- net Servo_PWM1: now also A1.14 (GPIO10)
- net Servo_PWM2: now also A1.15 (GPIO11)
- net Thermocouple_SCK: now also A1.4 (GPIO2); no longer A1.24 (GPIO18)
- net Thermocouple_SO: now also A1.1 (GPIO0); no longer A1.21 (GPIO16)
- net VIN: now also J1.2
- net at Q15.2 (D), Q16.1 (G), R21.2: now also Q3.1 (G)
- net at Q16.2 (D), R23.2: now also Q10.1 (G)
- net GPIO renamed Valve2
- net output_A renamed Valve2+
- net Valve2+: now also J9.1, Q3.2 (D)
- net output_B renamed Valve2-
- net Valve2-: now also J9.3, Q10.2 (D)
- new net: Q12.1 (G), Q20.2 (D), R39.2
- new net: Q19.2 (D), Q20.1 (G), Q5.1 (G), R37.2
- new net: Q11.1 (G), Q18.2 (D), R34.2
- new net: Q17.2 (D), Q18.1 (G), Q4.1 (G), R26.2
- new net Valve1: Q17.1 (G), R33.1
- new net Valve1+: J10.1, Q4.2 (D), R25.1
- new net Valve1-: J10.3, Q11.2 (D), R35.1
- new net Valve3: Q19.1 (G), R38.1
- new net Valve3+: J8.1, Q5.2 (D), R36.1
- new net Valve3-: J8.3, Q12.2 (D), R40.1
- no-connect marks 4 -> 3
Other:
- moved on the sheet: C33, C34, C35, C36, C37, C38, C39, C40, C41, J4, L4, Q15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

Commit message: Hydra v2 with html bom@
Connections:
- net GND: now also J4.3 (SHIELD1), J4.4 (SHIELD2); no longer J4.1, J4.2
- net RS485 DE/RE: now also A1.24 (GPIO18)
- net RS485_DI: now also A1.21 (GPIO16)
- net RS485_RO: now also A1.25 (GPIO19)
- net RS_A: now also J4.2; no longer J4.4 (SHIELD2)
- net RS_B: now also J4.1; no longer J4.3 (SHIELD1)
Other:
- moved on the sheet: J4

Commit message: changes
Parts:
- removed J1: XT30UPB-F, XT30UPB-F:XT30UPBF, symbol XT30UPB-F:XT30UPB-F
- removed J4: 1723103102, 1723103102:CONN02_1723103102_MOL, symbol 1723103102:1723103102
- added D1, D10, D2, D3, D8, D9: D_Schottky, symbol Device:D_Schottky
- added J11, J12, J7: 1723103103, 1723103103:MOLEX_1723103103, symbol 1723103103:1723103103
- added J2: 1200700164, CONN_1200700164_MOL, symbol 1200700164_MOL:1200700164
- added R41, R43: 4.7k, Resistor_SMD:R_0603_1608Metric_Pad0.98x0.95mm_HandSolder, symbol Device:R_Small
- added R42: 120, Resistor_SMD:R_0603_1608Metric_Pad0.98x0.95mm_HandSolder, symbol Device:R_Small
- C5: value C_Small -> 10uF
Connections:
- net Servo_GND is gone; now on net GND: J5.3, J6.3
- net +12V: now also R34.2, J11.1, J12.1, J2.1, J7.1; no longer R34.1
- net +3.3V: now also C4.1, C5.1, IC4.8 (VCC), R43.1
- net +5V: no longer C4.1, C5.1, IC4.8 (VCC)
- net ADC_A0: no longer U2.7 (A0)
- net ADC_A1: no longer U2.8 (A1)
- net ADC_A2: no longer U2.9 (A2)
- net GND: now also J6.S1 (SHIELD1), J6.S2 (SHIELD2), D1.2 (A), D10.2 (A), D2.2 (A), D3.2 (A), D8.2 (A), D9.2 (A), J11.3, J11.S1 (SHIELD1), J11.S2 (SHIELD2), J12.3, J12.S1 (SHIELD1), J12.S2 (SHIELD2), J2.2, J7.3, J7.S1 (SHIELD1), J7.S2 (SHIELD2), R41.2
- net RS_A: now also IC4.6 (A), J2.3, R42.1, R43.2; no longer IC4.7 (B)
- net RS_B: now also IC4.7 (B), J2.4, R41.1, R42.2; no longer IC4.6 (A)
- net Valve1+: now also D8.1 (K)
- net Valve1-: now also D3.1 (K)
- net Valve2+: now also D10.1 (K)
- net Valve2-: now also D9.1 (K)
- net Valve3+: now also D2.1 (K)
- net Valve3-: now also D1.1 (K)
- net at Q11.1 (G), Q18.2 (D): now also R34.1; no longer R34.2
- net ADC_A3: no longer names the net of U2.10 (A3)
- net RS485_DI renamed RS485_TX
- net RS485_RO renamed RS485_RX
- new net PRESSURE_1: J12.2, U2.7 (A0)
- new net PRESSURE_2: J11.2, U2.8 (A1)
- new net PRESSURE_3: J7.2, U2.9 (A2)
Other:
- note added: "Power and Data Connector"
- note added: "Pressure Transducers"
- note added: "Servo Connectors"
- note added: "would be good to separate grounds rafa doesnt know how"
- note removed: "Pressure Transducer ADC Amplifier"
- moved on the sheet: J5, J6, J8, R34, U2

Commit message: Hydra2
Connections:
- net RS_A: now also J2.4; no longer J2.3
- net RS_B: now also J2.3; no longer J2.4
