File: Boards/Avionics/HYDRA_V2/HYDRA_V2/HYDRA_V2.kicad_pcb (KiCad board)
At the start: 2 copper layers, 150.5 x 60.5 mm, 57 parts, among them IC1 MAX31855KASA+T, IC2 MAX31855KASA+T, IC3 MAX31855KASA+T, IC4 SP3485CN-L_TR, J4 1723103102, J5 1723103103, J6 1723103103, Q1 PMOS, Q14 PMOS, Q15 IRLB3813PBF-ND, Q16 IRLB3813PBF-ND, Q17 PMOS, Q2 IRLB3813PBF-ND, Q4 IRLB3813PBF-ND, Q5 PMOS, Q6 IRLB3813PBF-ND, Q7 PMOS, Q8 IRLB3813PBF-ND, Q9 PMOS, U3 ThermoConnector, U4 ThermoConnector, U5 ThermoConnector

Commit message: Hydra v2
Parts:
- removed U6, U7, U8: ~, DCDCModule:DCDC_Module
- added C10: 2.7nF, Capacitor_SMD:C_0603_1608Metric_Pad1.08x0.95mm_HandSolder, F.Cu at (95.5, 101.4)
- added C11: 22pF, Capacitor_SMD:C_0603_1608Metric_Pad1.08x0.95mm_HandSolder, F.Cu at (98.3, 97.8)
- added C12: 22uF, Capacitor_SMD:C_0603_1608Metric_Pad1.08x0.95mm_HandSolder, F.Cu at (87.8, 104.8)
- added C13: 22uF, Capacitor_SMD:C_0603_1608Metric_Pad1.08x0.95mm_HandSolder, F.Cu at (84.8, 104.8)
- added C14: 22uF, Capacitor_SMD:C_0603_1608Metric_Pad1.08x0.95mm_HandSolder, F.Cu at (81.8, 104.8)
- added C15: 10uF, Capacitor_SMD:C_0805_2012Metric_Pad1.18x1.45mm_HandSolder, F.Cu at (363.3, 55.8)
- added C16: 10nF, Capacitor_SMD:C_0603_1608Metric_Pad1.08x0.95mm_HandSolder, F.Cu at (363.1, 32.9)
- added C17: 2.7nF, Capacitor_SMD:C_0603_1608Metric_Pad1.08x0.95mm_HandSolder, F.Cu at (363.1, 35.4)
- added C18: 100nF, Capacitor_SMD:C_0603_1608Metric_Pad1.08x0.95mm_HandSolder, F.Cu at (363.1, 37.9)
- added C19: 47pF, Capacitor_SMD:C_0603_1608Metric_Pad1.08x0.95mm_HandSolder, F.Cu at (363.1, 40.4)
- added C20: 22pF, Capacitor_SMD:C_0603_1608Metric_Pad1.08x0.95mm_HandSolder, F.Cu at (363.1, 43.0)
- added C21: 22uF, Capacitor_SMD:C_0603_1608Metric_Pad1.08x0.95mm_HandSolder, F.Cu at (363.1, 45.5)
- added C22: 22uF, Capacitor_SMD:C_0603_1608Metric_Pad1.08x0.95mm_HandSolder, F.Cu at (363.1, 48.0)
- added C23: 22uF, Capacitor_SMD:C_0603_1608Metric_Pad1.08x0.95mm_HandSolder, F.Cu at (363.1, 50.5)
- added C24: 10uF, Capacitor_SMD:C_0805_2012Metric_Pad1.18x1.45mm_HandSolder, F.Cu at (363.3, 58.8)
- added C25: 10nF, Capacitor_SMD:C_0603_1608Metric_Pad1.08x0.95mm_HandSolder, F.Cu at (363.1, 53.0)
- added C26: 2.7nF, Capacitor_SMD:C_0603_1608Metric_Pad1.08x0.95mm_HandSolder, F.Cu at (367.4, 32.9)
- added C27: 100nF, Capacitor_SMD:C_0603_1608Metric_Pad1.08x0.95mm_HandSolder, F.Cu at (367.4, 35.4)
- added C28: 47pF, Capacitor_SMD:C_0603_1608Metric_Pad1.08x0.95mm_HandSolder, F.Cu at (367.4, 37.9)
- added C29: 22pF, Capacitor_SMD:C_0603_1608Metric_Pad1.08x0.95mm_HandSolder, F.Cu at (367.4, 40.4)
- added C30: 22uF, Capacitor_SMD:C_0603_1608Metric_Pad1.08x0.95mm_HandSolder, F.Cu at (367.4, 43.0)
- added C31: 22uF, Capacitor_SMD:C_0603_1608Metric_Pad1.08x0.95mm_HandSolder, F.Cu at (367.4, 45.5)
- added C32: 22uF, Capacitor_SMD:C_0603_1608Metric_Pad1.08x0.95mm_HandSolder, F.Cu at (367.4, 48.0)
- added C33: 10uF, Capacitor_SMD:C_0805_2012Metric_Pad1.18x1.45mm_HandSolder, F.Cu at (363.3, 61.8)
- added C34: 10nF, Capacitor_SMD:C_0603_1608Metric_Pad1.08x0.95mm_HandSolder, F.Cu at (367.4, 50.5)
- added C35: 2.7nF, Capacitor_SMD:C_0603_1608Metric_Pad1.08x0.95mm_HandSolder, F.Cu at (367.4, 53.0)
- added C36: 100nF, Capacitor_SMD:C_0603_1608Metric_Pad1.08x0.95mm_HandSolder, F.Cu at (371.8, 32.9)
- added C37: 47pF, Capacitor_SMD:C_0603_1608Metric_Pad1.08x0.95mm_HandSolder, F.Cu at (371.8, 35.4)
- added C38: 22pF, Capacitor_SMD:C_0603_1608Metric_Pad1.08x0.95mm_HandSolder, F.Cu at (371.8, 37.9)
- added C39: 22uF, Capacitor_SMD:C_0603_1608Metric_Pad1.08x0.95mm_HandSolder, F.Cu at (371.8, 40.4)
- added C40: 22uF, Capacitor_SMD:C_0603_1608Metric_Pad1.08x0.95mm_HandSolder, F.Cu at (371.8, 43.0)
- added C41: 22uF, Capacitor_SMD:C_0603_1608Metric_Pad1.08x0.95mm_HandSolder, F.Cu at (371.8, 45.5)
- added C6: 10uF, Capacitor_SMD:C_0805_2012Metric_Pad1.18x1.45mm_HandSolder, F.Cu at (96.1, 111.9)
- added C7: 10nF, Capacitor_SMD:C_0603_1608Metric_Pad1.08x0.95mm_HandSolder, F.Cu at (100.4, 108.8)
- added C8: 100nF, Capacitor_SMD:C_0603_1608Metric_Pad1.08x0.95mm_HandSolder, F.Cu at (92.7, 109.0)
- added C9: 47pF, Capacitor_SMD:C_0603_1608Metric_Pad1.08x0.95mm_HandSolder, F.Cu at (103.2, 103.5)
- added D7: LED, LED_THT:LED_D3.0mm, F.Cu at (155.3, 160.2)
- added L1: 6.8uH, SPM10054T-6R8M-HZR:SPM10054T6R8MHZR, F.Cu at (85.3, 96.8)
- added L2: 6.8uH, SPM10054T-6R8M-HZR:SPM10054T6R8MHZR, F.Cu at (352.5, 38.2)
- added L3: 6.8uH, SPM10054T-6R8M-HZR:SPM10054T6R8MHZR, F.Cu at (352.5, 51.3)
- added L4: 6.8uH, SPM10054T-6R8M-HZR:SPM10054T6R8MHZR, F.Cu at (352.5, 64.4)
- added R12: 62, Resistor_SMD:R_0805_2012Metric, F.Cu at (175.2, 164.2)
- added R13: 27kO, Resistor_SMD:R_0603_1608Metric_Pad0.98x0.95mm_HandSolder, F.Cu at (98.3, 101.5)
- added R14: 210kO, Resistor_SMD:R_0603_1608Metric_Pad0.98x0.95mm_HandSolder, F.Cu at (100.4, 101.9)
- added R18: 22.1kO, Resistor_SMD:R_0603_1608Metric_Pad0.98x0.95mm_HandSolder, F.Cu at (100.4, 105.4)
- added R19: 27kO, Resistor_SMD:R_0603_1608Metric_Pad0.98x0.95mm_HandSolder, F.Cu at (371.8, 48.0)
- added R25: 69.8kO, Resistor_SMD:R_0603_1608Metric_Pad0.98x0.95mm_HandSolder, F.Cu at (371.8, 50.5)
- added R26: 22.1kO, Resistor_SMD:R_0603_1608Metric_Pad0.98x0.95mm_HandSolder, F.Cu at (371.8, 53.0)
- added R27: 27kO, Resistor_SMD:R_0603_1608Metric_Pad0.98x0.95mm_HandSolder, F.Cu at (376.1, 32.9)
- added R28: 210kO, Resistor_SMD:R_0603_1608Metric_Pad0.98x0.95mm_HandSolder, F.Cu at (376.1, 35.4)
- added R29: 22.1kO, Resistor_SMD:R_0603_1608Metric_Pad0.98x0.95mm_HandSolder, F.Cu at (376.1, 37.9)
- added R30: 27kO, Resistor_SMD:R_0603_1608Metric_Pad0.98x0.95mm_HandSolder, F.Cu at (376.1, 40.4)
- added R31: 210kO, Resistor_SMD:R_0603_1608Metric_Pad0.98x0.95mm_HandSolder, F.Cu at (376.1, 43.0)
- added R32: 22.1kO, Resistor_SMD:R_0603_1608Metric_Pad0.98x0.95mm_HandSolder, F.Cu at (376.1, 45.5)
- added U1: AP64501SP-13, AP64501SP_13:SOP_AP64501SP-13_DIO, F.Cu at (96.6, 106.9)
- added U10: AP64501SP-13, AP64501SP_13:SOP_AP64501SP-13_DIO, F.Cu at (382.5, 34.9)
- added U11: AP64501SP-13, AP64501SP_13:SOP_AP64501SP-13_DIO, F.Cu at (382.5, 41.5)
- added U12: AP64501SP-13, AP64501SP_13:SOP_AP64501SP-13_DIO, F.Cu at (382.5, 48.1)
- IC1, IC2, IC3: moved to B.Cu
- Q1, Q14, Q17, Q5, Q7, Q9: footprint Package_TO_SOT_THT:TO-220-3_Vertical -> STD46P4LLF6:STD46P4LLF6
- Q15, Q16, Q2, Q4, Q6, Q8: footprint Package_TO_SOT_THT:TO-220-3_Vertical -> Package_TO_SOT_SMD:SOT-223
- moved IC1 245.9 mm to (92.5, 63.2), turned to 90 degrees
- moved IC2 228.2 mm to (110.2, 63.2), turned to 90 degrees
- moved IC3 211.1 mm to (127.4, 63.2), turned to 90 degrees
- moved IC4 208.3 mm to (131.3, 100.1)
- moved R1 141.0 mm to (389.1, 33.1)
- moved R2 141.0 mm to (389.1, 36.1)
- moved R3 141.0 mm to (389.1, 39.0)
- moved R4 141.0 mm to (389.1, 42.0)
- moved Q17 137.2 mm to (387.1, 24.2)
- moved R11 131.3 mm to (389.1, 44.9)
- moved Q9 130.8 mm to (367.9, 24.2)
- moved R22 125.7 mm to (389.1, 47.9)
- moved Q5 124.6 mm to (348.7, 24.2)
- moved Q14 119.8 mm to (377.5, 24.2)
- moved Q7 116.2 mm to (358.3, 24.2)
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Connections:
- D5 pad 2: +5V -> Servo_VCC
- D6 pad 2: +3.3V -> +5V
Routing:
- net Servo_VCC: track 0.00 -> 33.2 mm, vias 0 -> 2
- net Net-(U1-SW): track 0.00 -> 18.2 mm
- net Net-(U1-COMP): track 0.00 -> 6.76 mm
- net Net-(U1-FB): track 0.00 -> 6.44 mm
- net VIN: track 0.00 -> 3.82 mm
- net GND: track 0.00 -> 2.90 mm, vias 0 -> 9
- net Net-(C10-Pad1): track 0.00 -> 2.85 mm
- net Net-(U1-SS): track 0.00 -> 1.95 mm
Other:
- copper layers 2 -> 4

Commit message: Hydra v2 almost done
Parts:
- removed C15: 10uF, Capacitor_SMD:C_0805_2012Metric_Pad1.18x1.45mm_HandSolder
- removed C16: 10nF, Capacitor_SMD:C_0603_1608Metric_Pad1.08x0.95mm_HandSolder
- removed C17: 2.7nF, Capacitor_SMD:C_0603_1608Metric_Pad1.08x0.95mm_HandSolder
- removed C18: 100nF, Capacitor_SMD:C_0603_1608Metric_Pad1.08x0.95mm_HandSolder
- removed C19: 47pF, Capacitor_SMD:C_0603_1608Metric_Pad1.08x0.95mm_HandSolder
- removed C20: 22pF, Capacitor_SMD:C_0603_1608Metric_Pad1.08x0.95mm_HandSolder
- removed C21, C22, C23: 22uF, Capacitor_SMD:C_0603_1608Metric_Pad1.08x0.95mm_HandSolder
- removed L2: 6.8uH, SPM10054T-6R8M-HZR:SPM10054T6R8MHZR
- removed Q1, Q14, Q7, Q9: PMOS, STD46P4LLF6:STD46P4LLF6
- removed Q2, Q6, Q8: IRLB3813PBF-ND, Package_TO_SOT_SMD:SOT-223
- removed R1, R10, R11, R15, R16, R17, R2, R3, R4, R9: 10K, Resistor_SMD:R_0805_2012Metric_Pad1.20x1.40mm_HandSolder
- removed R19: 27kO, Resistor_SMD:R_0603_1608Metric_Pad0.98x0.95mm_HandSolder
- removed U10: AP64501SP-13, AP64501SP_13:SOP_AP64501SP-13_DIO
- added J1: XT30UPB-F, XT30UPB-F:XT30UPBF, F.Cu at (204.2, 58.8)
- added J10: 1723103103, 1723103103:MOLEX_1723103103, F.Cu at (202.4, 101.3)
- added J8: 1723103103, 1723103103:MOLEX_1723103103, F.Cu at (185.6, 101.3)
- added J9: 1723103103, 1723103103:MOLEX_1723103103, F.Cu at (147.6, 67.1)
- added Q10: STD46P4LLF6, STD46P4LLF6:STD46P4LLF6, F.Cu at (122.0, 95.5)
- added Q11: STD46P4LLF6, STD46P4LLF6:STD46P4LLF6, F.Cu at (222.1, 85.3)
- added Q12: STD46P4LLF6, STD46P4LLF6:STD46P4LLF6, F.Cu at (131.7, 110.2)
- added Q18: IRLB3813PBF-ND, Package_TO_SOT_SMD:SOT-223, F.Cu at (222.3, 96.5)
- added Q19: IRLB3813PBF-ND, Package_TO_SOT_SMD:SOT-223, F.Cu at (190.6, 86.1)
- added Q20: IRLB3813PBF-ND, Package_TO_SOT_SMD:SOT-223, F.Cu at (149.7, 110.3)
- added Q3: STD46P4LLF6, STD46P4LLF6:STD46P4LLF6, F.Cu at (139.7, 83.7)
- added R33: 10K, Resistor_SMD:R_0805_2012Metric_Pad1.20x1.40mm_HandSolder, F.Cu at (216.8, 101.8)
- added R34: 10K, Resistor_SMD:R_0805_2012Metric_Pad1.20x1.40mm_HandSolder, F.Cu at (216.8, 90.4)
- added R35: 10K, Resistor_SMD:R_0805_2012Metric_Pad1.20x1.40mm_HandSolder, F.Cu at (225.4, 77.1)
- added R36: 10K, Resistor_SMD:R_0805_2012Metric_Pad1.20x1.40mm_HandSolder, F.Cu at (144.0, 93.5)
- added R37: 10K, Resistor_SMD:R_0805_2012Metric_Pad1.20x1.40mm_HandSolder, F.Cu at (190.7, 90.8)
- added R38: 10K, Resistor_SMD:R_0805_2012Metric_Pad1.20x1.40mm_HandSolder, F.Cu at (184.9, 87.2)
- added R39: 10K, Resistor_SMD:R_0805_2012Metric_Pad1.20x1.40mm_HandSolder, F.Cu at (155.2, 112.0)
- added R40: 10K, Resistor_SMD:R_0805_2012Metric_Pad1.20x1.40mm_HandSolder, F.Cu at (193.6, 94.0)
- C1, C10, C11, C12, C13, C14, C2, C24, C25, C26, C27, C28, C3, C30, C31, C32, C33, C34, C35, C36, C37, C39, C40, C41, C6, C7, C8, C9, L1, L3, L4, R13, R14, R18, R29, R32, U1, U11, U12: moved to B.Cu
- C29: value 22pF -> 33pF; moved to B.Cu
- C38: value 22pF -> 15pF; moved to B.Cu
- D4, D5, D6, D7: footprint LED_THT:LED_D3.0mm -> LED-Yellow_VLMY1300-GS08:LEDC1608X100N
- Q17: value PMOS -> IRLB3813PBF-ND; footprint STD46P4LLF6:STD46P4LLF6 -> Package_TO_SOT_SMD:SOT-223
- Q4: value IRLB3813PBF-ND -> STD46P4LLF6; footprint Package_TO_SOT_SMD:SOT-223 -> STD46P4LLF6:STD46P4LLF6
- Q5: value PMOS -> STD46P4LLF6
- R25: value 69.8kO -> 10K; footprint Resistor_SMD:R_0603_1608Metric_Pad0.98x0.95mm_HandSolder -> Resistor_SMD:R_0805_2012Metric_Pad1.20x1.40mm_HandSolder
- R26: value 22.1kO -> 10K; footprint Resistor_SMD:R_0603_1608Metric_Pad0.98x0.95mm_HandSolder -> Resistor_SMD:R_0805_2012Metric_Pad1.20x1.40mm_HandSolder
- R27: value 27kO -> 15.8kO; moved to B.Cu
- R28: value 210kO -> 115.8kO; moved to B.Cu
- R30: value 27kO -> 37.4kO; moved to B.Cu
- R31: value 210kO -> 309kO; moved to B.Cu
- moved R22 267.7 mm to (124.3, 87.5)
- moved R8 260.4 mm to (78.8, 81.2), turned to 180 degrees
- moved R7 259.3 mm to (78.9, 86.2), turned to 180 degrees
- moved R6 258.5 mm to (78.8, 91.2), turned to 180 degrees
- moved U12 254.0 mm to (133.3, 97.5), turned to -90 degrees
- moved D6 253.6 mm to (82.6, 81.2)
- moved D4 253.3 mm to (82.6, 91.2)
- moved D5 253.2 mm to (82.6, 86.2)
- moved C36 250.7 mm to (129.7, 97.7), turned to -90 degrees
- moved C1 250.5 mm to (87.9, 67.0)
- moved R30 248.9 mm to (135.2, 103.0), turned to -90 degrees
- moved R32 244.9 mm to (137.8, 102.1)
- moved R31 244.4 mm to (137.8, 97.3), turned to 180 degrees
- moved C38 243.4 mm to (137.8, 105.0)
- moved C37 242.8 mm to (137.8, 100.3), turned to 180 degrees
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Connections:
- A1 pad 1: unconnected-(A1-GPIO0-Pad1) -> Thermocouple_SO
- A1 pad 14: unconnected-(A1-GPIO10-Pad14) -> Servo_PWM1
- A1 pad 15: unconnected-(A1-GPIO11-Pad15) -> Servo_PWM2
- A1 pad 21: Thermocouple_SO -> unconnected-(A1-GPIO16-Pad21)
- A1 pad 24: Thermocouple_SCK -> unconnected-(A1-GPIO18-Pad24)
- A1 pad 36: unconnected-(A1-3V3-Pad36)_1 -> +3.3V
- A1 pad 4: unconnected-(A1-GPIO2-Pad4) -> Thermocouple_SCK
- C28 pad 1: Net-(C28-Pad1) -> +5V
- C30 pad 1: Net-(C28-Pad1) -> +5V
- C31 pad 1: Net-(C28-Pad1) -> +5V
- C32 pad 1: Net-(C28-Pad1) -> +5V
- C37 pad 1: Net-(C37-Pad1) -> +12V
- C39 pad 1: Net-(C37-Pad1) -> +12V
- C40 pad 1: Net-(C37-Pad1) -> +12V
- C41 pad 1: Net-(C37-Pad1) -> +12V
- J4 pad 3: RS_A -> RS_B
- J4 pad 4: RS_B -> RS_A
- L3 pad 2: Net-(C28-Pad1) -> +5V
- L4 pad 2: Net-(C37-Pad1) -> +12V
- Q15 pad 1: GPIO -> Valve2
- Q16 pad 2: Net-(Q16-D) -> Net-(Q10-G)
- Q17 pad 1: output_B -> Valve1
- Q17 pad 2: Net-(Q16-D) -> Net-(Q17-D)
- Q17 pad 3: +12V -> GND
- Q4 pad 1: GPIO -> Net-(Q17-D)
- Q4 pad 2: Net-(Q4-D) -> Valve1+
- Q4 pad 3: GND -> +12V
- Q5 pad 1: output_A -> Net-(Q19-D)
- Q5 pad 2: Net-(Q4-D) -> Valve3+
- R20 pad 1: output_A -> Valve2+
- R22 pad 1: GPIO -> Valve2
- R23 pad 2: Net-(Q16-D) -> Net-(Q10-G)
- R24 pad 1: output_B -> Valve2-
- R25 pad 1: Net-(C19-Pad1) -> Valve1+
- R25 pad 2: Net-(U10-FB) -> GND
- R26 pad 1: Net-(U10-FB) -> +12V
- R26 pad 2: GND -> Net-(Q17-D)
- R28 pad 1: Net-(C28-Pad1) -> +5V
- R31 pad 1: Net-(C37-Pad1) -> +12V
Routing:
- net +12V: track 0.00 -> 281.9 mm, vias 0 -> 6
- net +5V: track 0.00 -> 222.0 mm, vias 0 -> 5
- net Thermocouple_CS1: track 0.00 -> 122.7 mm, vias 0 -> 1
- net GND: track 2.90 -> 123.8 mm, vias 9 -> 64
- net Thermocouple_SO: track 0.00 -> 114.9 mm
- net +3.3V: track 0.00 -> 108.0 mm, vias 0 -> 1
- net Servo_PWM2: track 0.00 -> 83.4 mm, vias 0 -> 1
- net Thermocouple_SCK: track 0.00 -> 76.0 mm, vias 0 -> 4
- net Valve3-: track 0.00 -> 74.0 mm
- net Net-(Q19-D): track 0.00 -> 69.7 mm
- net Servo_PWM1: track 0.00 -> 69.5 mm
- net Valve3+: track 0.00 -> 51.7 mm
- net Thermocouple_CS2: track 0.00 -> 50.5 mm, vias 0 -> 1
- net Servo_VCC: track 33.2 -> 80.1 mm, vias 2 -> 3
- net Valve2-: track 0.00 -> 45.4 mm
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- added copper zone on B.Cu, net VIN
Other:
- board size 150.5 x 60.5 mm -> 151 x 61 mm
- copper layers 4 -> 2
- board text added: "12V"
- board text added: "3V3"
- board text added: "5V"
- board text added: "8V4"

Commit message: Hydra v2 with html bom@
Parts:
- moved R38 3.51 mm to (187.3, 89.7)
- moved R37 3.41 mm to (189.7, 94.0)
- moved Q19 2.94 mm to (192.8, 88.0)
- moved R40 1.84 mm to (195.4, 94.0)
- moved IC4 0.36 mm to (213.9, 74.5)
Connections:
- A1 pad 21: unconnected-(A1-GPIO16-Pad21) -> RS485_DI
- A1 pad 24: unconnected-(A1-GPIO18-Pad24) -> RS485 DE/RE
- A1 pad 25: unconnected-(A1-GPIO19-Pad25) -> RS485_RO
- J4 pad 1: GND -> RS_B
- J4 pad 2: GND -> RS_A
- J4 pad 3: RS_B -> GND
- J4 pad 4: RS_A -> GND
Routing:
- net RS485_DI: track 0.00 -> 55.8 mm, vias 0 -> 2
- net RS485 DE/RE: track 1.98 -> 49.4 mm
- net RS485_RO: track 0.00 -> 44.4 mm
- net GND: track 123.8 -> 139.4 mm
- net RS_B: track 15.6 -> 5.05 mm
- net RS_A: track 15.2 -> 5.06 mm
- net +12V: track 281.9 -> 284.3 mm
- net Net-(Q19-D): track 69.7 -> 67.9 mm
- net Valve3-: track 74.0 -> 74.8 mm
- net Valve3: track 3.44 -> 4.01 mm

Commit message: Hydra2
Parts:
- removed J4: 1723103102, 1723103102:CONN02_1723103102_MOL
- added D11: SS10PH102HM3_I, SS10PH102HM3_I:SS10PH102HM3I, F.Cu at (150.5, 87.3)
- added D12: SS10PH102HM3_I, SS10PH102HM3_I:SS10PH102HM3I, F.Cu at (121.5, 109.0)
- added D13: SS10PH102HM3_I, SS10PH102HM3_I:SS10PH102HM3I, F.Cu at (119.0, 80.5)
- added D14: SS10PH102HM3_I, SS10PH102HM3_I:SS10PH102HM3I, F.Cu at (150.5, 78.2)
- added D15: SS10PH102HM3_I, SS10PH102HM3_I:SS10PH102HM3I, F.Cu at (176.2, 111.2)
- added D16: SS10PH102HM3_I, SS10PH102HM3_I:SS10PH102HM3I, F.Cu at (215.2, 57.5)
- added J11: 1723103103, 1723103103:MOLEX_1723103103, B.Cu at (151.6, 131.1)
- added J12: 1723103103, 1723103103:MOLEX_1723103103, B.Cu at (203.0, 37.0)
- added J7: 1723103103, 1723103103:MOLEX_1723103103, B.Cu at (169.0, 131.1)
- added R41: 4.7k, Resistor_SMD:R_0603_1608Metric_Pad0.98x0.95mm_HandSolder, F.Cu at (198.0, 62.5)
- added R42: 120, Resistor_SMD:R_0603_1608Metric_Pad0.98x0.95mm_HandSolder, F.Cu at (201.6, 62.5)
- added R43: 4.7k, Resistor_SMD:R_0603_1608Metric_Pad0.98x0.95mm_HandSolder, F.Cu at (205.1, 62.5)
- C5: value C_Small -> 10uF
- J1: value XT30UPB-F -> 1723163304; footprint XT30UPB-F:XT30UPBF -> 1723163304:MOLEX_1723163304
- moved C4 12.5 mm to (198.0, 69.3)
- moved C5 12.5 mm to (198.0, 65.8)
- moved IC4 12.5 mm to (203.0, 68.5)
- moved J1 12.2 mm to (210.5, 69.2)
- turned R34 to 90 degrees
Connections:
- net RS485_DI renamed RS485_TX
- net RS485_RO renamed RS485_RX
- net Servo_VCC renamed +8.4V
- C4 pad 1: +5V -> +3.3V
- C5 pad 1: +5V -> +3.3V
- IC4 pad 6: RS_B -> RS_A
- IC4 pad 7: RS_A -> RS_B
- IC4 pad 8: +5V -> +3.3V
- J1 pad 1: GND -> +12V
- J1 pad 2: VIN -> RS_A
- J5 pad 3: Servo_GND -> GND
- J6 pad 3: Servo_GND -> GND
- J6 pad S1: unconnected-(J6-SHIELD1-PadS1) -> GND
- J6 pad S2: unconnected-(J6-SHIELD2-PadS2) -> GND
- R34 pad 1: +12V -> Net-(Q11-G)
- R34 pad 2: Net-(Q11-G) -> +12V
- U2 pad 10: ADC_A3 -> unconnected-(U2-A3-Pad10)
- U2 pad 7: ADC_A0 -> PRESSURE_1
- U2 pad 8: ADC_A1 -> PRESSURE_2
- U2 pad 9: ADC_A2 -> PRESSURE_3
Routing:
- net +3.3V: track 108.0 -> 149.2 mm, vias 1 -> 3
- net Valve1+: track 18.1 -> 55.5 mm, vias 0 -> 2
- net GND: track 139.4 -> 170.3 mm
- net Valve1-: track 29.4 -> 58.6 mm
- net ADC_A1: track 23.9 -> 0.92 mm
- net ADC_A0: track 23.9 -> 1.13 mm
- net ADC_A2: track 22.8 -> 1.05 mm
- net +12V: track 284.3 -> 305.5 mm, vias 6 -> 8
- net Servo_GND: track 20.0 -> 0.00 mm
- net RS_B: track 5.05 -> 19.6 mm
- net +5V: track 222.0 -> 210.0 mm
- net Valve3+: track 51.7 -> 60.9 mm
- net Valve3-: track 74.8 -> 83.9 mm
- net RS_A: track 5.06 -> 14.0 mm
- net RS485_TX: track 55.8 -> 64.7 mm
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