File: Boards/Avionics/HYDRA_V2/HYDRA_V2/_restore_backup_2026-07-01T21-53-16-686/HYDRA_V2.kicad_sch (KiCad schematic)
At the start: 57 parts, among them IC1 MAX31855KASA+T, IC2 MAX31855KASA+T, IC3 MAX31855KASA+T, IC4 SP3485CN-L_TR, J4 1723103102, J5 1723103103, J6 1723103103, Q1 PMOS, Q14 PMOS, Q15 IRLB3813PBF-ND, Q16 IRLB3813PBF-ND, Q17 PMOS, Q2 IRLB3813PBF-ND, Q4 IRLB3813PBF-ND, Q5 PMOS, Q6 IRLB3813PBF-ND, Q7 PMOS, Q8 IRLB3813PBF-ND, Q9 PMOS, U3 ThermoConnector, U4 ThermoConnector, U5 ThermoConnector

Commit message: Hydra v2
Parts:
- U2, U6, U7, U8: value ~ -> (none)
