File: Boards/Avionics/CORTEX/CORTEX_ALPHA/CORTEX_ALPHA.kicad_sch (KiCad schematic)
At the start: 15 parts, among them J1 Conn_01x06_Pin, J2 Screw_Terminal_01x02, J3 1200700164, J4 Conn_01x06_Pin, U2 E28-2G4M27S_LoRa, U3 MAX485_MODULE_5V_LOGIC_TLL_TO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, U4 NUCLEO-G431KB

Commit message: changes cortex
Parts:
- removed CanBus_Module1: ~, CORTEX:Canbus, symbol CanBus:MCP2551_Module
- removed J2: Screw_Terminal_01x02, TerminalBlock:TerminalBlock_Xinya_XY308-2.54-2P_1x02_P2.54mm_Horizontal, symbol Connector:Screw_Terminal_01x02
- removed U3: MAX485_MODULE_5V_LOGIC_TLL_TO_RS-485_CONVERTER, MAX485_MODULE_5V_LOGIC_TLL_TO_RS-485_CONVERTER:MODULE_MAX485_MODULE_5V_LOGIC_TLL_TO_RS-485_CONVERTER, symbol MAX485_MODULE_5V_LOGIC_TLL_TO_RS-485_CONVERTER:MAX485_MODULE_5V_LOGIC_TLL_TO_RS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
- removed U4: NUCLEO-G431KB, NUCLEO_G431KB:MODULE_NUCLEO-G431KB, symbol NUCLEO-G431KB:NUCLEO-G431KB
- added A1: RaspberryPi_Pico, Module:RaspberryPi_Pico_Common_Unspecified, symbol MCU_Module:RaspberryPi_Pico
- added C7: 0.1uF, Capacitor_SMD:C_0805_2012Metric, symbol Device:C_Small
- added C8: C_Small, Capacitor_SMD:C_0805_2012Metric, symbol Device:C_Small
- added IC5: SP3485CN-L_TR, Package_SO:SOIC-8_3.9x4.9mm_P1.27mm, symbol SP3485CN-L_TR:SP3485CN-L_TR
- added U1: LD1117S33TR_SOT223, Package_TO_SOT_SMD:SOT-223-3_TabPin2, symbol Regulator_Linear:LD1117S33TR_SOT223
- U5: value ~ -> (none)
Connections:
- net +3.3V: now also U1.2 (VO)
- net +5V: now also A1.39 (VSYS), C7.1, C8.1, IC5.8 (VCC), U1.3 (VI)
- net ANT_BUSY: now also A1.12 (GPIO9)
- net ANT_DIO1: now also A1.11 (GPIO8)
- net ANT_NRESET: now also A1.14 (GPIO10)
- net ANT_RX_EN: now also A1.9 (GPIO6)
- net ANT_TX_EN: now also A1.10 (GPIO7)
- net CLK: now also A1.4 (GPIO2)
- net GND: now also A1.13 (GND), A1.18 (GND), A1.23 (GND), A1.28 (GND), A1.3 (GND), A1.38 (GND), A1.8 (GND), C7.2, C8.2, IC5.5 (GND), U1.1 (GND)
- net MISO: now also A1.6 (GPIO4)
- net MOSI: now also A1.5 (GPIO3)
- net NAV CTS UART: now also A1.24 (GPIO18)
- net NAV RTS UART: now also A1.25 (GPIO19)
- net NAV RX UART: now also A1.22 (GPIO17)
- net NAV TX UART: now also A1.21 (GPIO16)
- net RS_A: now also IC5.6 (A)
- net RS_B: now also IC5.7 (B)
- net RS_ENABLE: now also A1.17 (GPIO13), IC5.2 (~{RE}), IC5.3 (DE)
- net RS_RX: now also A1.16 (GPIO12), IC5.1 (RO)
- net RS_TX: now also A1.15 (GPIO11), IC5.4 (DI)
- net CS renamed RADIO_CS
- net RADIO_CS: now also A1.7 (GPIO5); no longer J1.2 (Pin_2)
- new net SD_CS: A1.2 (GPIO1), J1.2 (Pin_2)
- no-connect marks 17 -> 2
Other:
- note added: "LDO 5V-3.3V"
- note added: "RADIO"
- note added: "RASPBERRY PI PICO"
- note removed: "ANTENNA"
- note removed: "CANBUS MODULE"
- note removed: "STM32 NUCLEO"
- moved on the sheet: C1, C2, C3, C4, R1, U5

Commit message: layout cortex new
Parts:
- added D1: D_Schottky, Diode_THT:D_A-405_P7.62mm_Horizontal, symbol Device:D_Schottky
Connections:
- net +5V: now also D1.1 (K); no longer C1.1, C2.1, U5.3 (OUT+)
- new net: C1.1, C2.1, D1.2 (A), U5.3 (OUT+)
Changed lines of the file:
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@@
 	)
 	(junction
-		(at 152.4 130.81)
+		(at 93.98 156.21)
 		(diameter 0)
 		(color 0 0 0 0)
 	)
 	(junction
-		(at 93.98 156.21)
+		(at 152.4 130.81)
 		(diameter 0)
 		(color 0 0 0 0)
@@
 	(wire
 		(pts
+			(xy 101.6 156.21) (xy 93.98 156.21)
+		)
+		(stroke
+			(width 0)
+			(type default)
+		)
+	)
+	(wire
+		(pts
 			(xy 146.05 135.89) (xy 148.59 135.89)
 		)
@@
 		)
 	)
+	(wire
+		(pts
+			(xy 111.76 156.21) (xy 111.76 154.94)
+		)
+		(stroke
+			(width 0)
+			(type default)
+		)
+	)
+	(wire
+		(pts
+			(xy 109.22 156.21) (xy 111.76 156.21)
+		)
+		(stroke
+			(width 0)
+			(type default)
+		)
+	)
 	(bus
 		(pts
@@
 	(wire
 		(pts
-			(xy 93.98 156.21) (xy 99.06 156.21)
-		)
-		(stroke
-			(width 0)
-			(type default)
-		)
-	)
-	(wire
-		(pts
 			(xy 148.59 133.35) (xy 152.4 133.35)
 		)
@@
 	(symbol
 		(lib_id "power:+5V")
-		(at 99.06 156.21 0)
+		(at 111.76 154.94 0)
 		(unit 1)
 		(body_style 1)
@@
 		(fields_autoplaced yes)
 		(property "Reference" "#PWR02"
-			(at 99.06 160.02 0)
+			(at 111.76 158.75 0)
 			(hide yes)
 			(show_name no)
@@
 		)
 		(property "Value" "+5V"
-			(at 99.06 151.13 0)
+			(at 111.76 149.86 0)
 			(show_name no)
 			(do_not_autoplace no)
@@
 		)
 		(property "Footprint" ""
-			(at 99.06 156.21 0)
+			(at 111.76 154.94 0)
 			(hide yes)
 			(show_name no)
@@
 		)
 		(property "Datasheet" ""
-			(at 99.06 156.21 0)
+			(at 111.76 154.94 0)
 			(hide yes)
 			(show_name no)
@@
 		)
 		(property "Description" "Power symbol creates a global label with name \"+5V\""
-			(at 99.06 156.21 0)
+			(at 111.76 154.94 0)
 			(hide yes)
 			(show_name no)
@@
 					(unit 1)
 				)
+			)
+		)
+	)
+	(symbol
+		(lib_id "Device:D_Schottky")
+		(at 105.41 156.21 180)
+		(unit 1)
+		(body_style 1)
+		(exclude_from_sim no)
+		(in_bom yes)
+		(on_board yes)
+		(in_pos_files yes)
+		(dnp no)
+		(fields_autoplaced yes)
+		(property "Reference" "D1"
+			(at 105.7275 149.86 0)
+			(show_name no)
+			(do_not_autoplace no)
+			(effects
+				(font
+					(size 1.27 1.27)
+				)
+			)
+		)
+		(property "Value" "D_Schottky"
+			(at 105.7275 152.4 0)
+			(show_name no)
+			(do_not_autoplace no)
+			(effects
+				(font
+					(size 1.27 1.27)
+				)
+			)
+		)
+		(property "Footprint" "Diode_THT:D_A-405_P7.62mm_Horizontal"
+			(at 105.41 156.21 0)
+			(hide yes)
+			(show_name no)
+			(do_not_autoplace no)
+			(effects
+				(font
+					(size 1.27 1.27)
+				)
+			)
+		)
+		(property "Datasheet" ""
+			(at 105.41 156.21 0)
+			(hide yes)
+			(show_name no)
+			(do_not_autoplace no)
+			(effects
+				(font
+					(size 1.27 1.27)
+				)
+			)
+		)
+		(property "Description" "Schottky diode"
+			(at 105.41 156.21 0)
+			(hide yes)
+			(show_name no)
+			(do_not_autoplace no)
+			(effects
+				(font
+					(size 1.27 1.27)
+				)
+			)
+		)
+		(pin "2"
+		)
+		(pin "1"
+		)
+		(instances
+			(project "CORTEX_ALPHA"
+				(path "/b3433ded-bc33-4d30-8ca0-59a8e98dfeda"
+					(reference "D1")
+					(unit 1)
+				)

Commit message: changes
Parts:
- removed C7: 0.1uF, Capacitor_SMD:C_0805_2012Metric, symbol Device:C_Small
- removed C8: C_Small, Capacitor_SMD:C_0805_2012Metric, symbol Device:C_Small
- removed R1: 1K, Resistor_SMD:R_0603_1608Metric_Pad0.98x0.95mm_HandSolder, symbol Device:R
- added C5: 47uF, symbol Device:C_Small
- added C6: 10uF, symbol Device:C_Small
- added R4: 120, symbol Device:R_Small
- added R5, R6: 4.7k, symbol Device:R_Small
- D1: footprint Diode_THT:D_A-405_P7.62mm_Horizontal -> (none)
Connections:
- net +3.3V: now also IC5.8 (VCC), C5.2, C6.2, R6.2
- net +5V: now also C1.1, C2.1, D1.2 (A), U5.3 (OUT+); no longer A1.39 (VSYS), D1.1 (K), IC5.8 (VCC), U1.3 (VI)
- net GND: now also C5.1, C6.1, R5.1
- net RS_A: now also R4.2, R6.1
- net RS_B: now also R4.1, R5.2
- new net +4.6V: A1.39 (VSYS), D1.1 (K), U1.3 (VI)
Other:
- note added: "navigator only works on batteries"
- note added: "only 4.6 if powered from batteries 5 if usb connected"

Commit message: Hydra2
Other:
- note added: "check if navigator needs 5, if not change to 4.6"
Changed lines of the file:
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@@
 	(generator_version "10.0")
 	(paper "A4")
+	(text "check if navigator needs 5, if not change to 4.6\n"
+		(exclude_from_sim no)
+		(at 312.42 59.436 0)
+		(effects
+			(font
+				(size 1.27 1.27)
+			)
+		)
+	)
 	(text "LDO 5V-3.3V\n"
 		(exclude_from_sim no)
@@
 	(wire
 		(pts
-			(xy 157.48 38.1) (xy 157.48 43.18)
-		)
-		(stroke
-			(width 0)
-			(type default)
-		)
-	)
-	(wire
-		(pts
 			(xy 254 137.16) (xy 252.73 137.16)
 		)
@@
 	(wire
 		(pts
-			(xy 132.08 38.1) (xy 157.48 38.1)
+			(xy 132.08 43.18) (xy 157.48 43.18)
 		)
 		(stroke
@@
 		)
 		(stroke
+			(width 0)
+			(type default)
+		)
+	)
+	(wire
+		(pts
+			(xy 132.08 43.18) (xy 132.08 38.1)
+		)
+		(stroke
